File: microdust_pcb/microdust_pcb/microdust_pcb.sch (KiCad schematic (older format))
At the start: 17 parts

Commit message: update
Parts:
- added C?: 0.1uF, symbol Device:C
- added J?: Conn_01x07, symbol Connector_Generic:Conn_01x07
- R?: footprint (none) -> Resistor_SMD:R_0603_1608Metric_Pad1.05x0.95mm_HandSolder
Connections:
- net labels added: CH_B, CS, DC, FAN, INPUT_B, RES
- wire segments 103 -> 121
Other:
- note added: "ISP Socket"
- note added: "OLED 128x64 I2C / SPI Connector"
- note added: "PMS7003 Micro Dust Sensor"
- note added: "Power Input LED Indicator"
- moved on the sheet: C?, D?, J?, R?, U?, Y?
